Commit message: [Integ] integration map, gui, central node

File: multitb_ws/src/turtlebot3_multi_robot/urdf/turtlebot3_waffle.urdf (robot description, URDF)
Before this commit: robot turtlebot3_waffle, 15 links, 14 joints
Links:
- removed link mounting_cylinder
- removed link mounting_plate
Joints:
- removed joint cylinder_rotation_joint
- removed joint cylinder_vertical_joint
